File: Hardware/CAD-eagle/TTE/prototype_total_schematic_2355_Depricated.brd (EAGLE design)
At the start: 100 x 80 mm, 24 parts, among them J2 MOLEX_48037-0001MOLEX_48037-0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, U1 LTC1069-7CS8#PBF, U2 FT232RL-BASICSSOP

Commit message: MODEM Files
Parts:
- removed C13: 100nF, SparkFun-Capacitors:0805
- removed C14: 22uF, SparkFun-Capacitors:0805
- removed C15: 470n, SparkFun-Capacitors:0805
- removed C16: 100n, SparkFun-Capacitors:0805
- removed C17: 1000p, SparkFun-Capacitors:0805
- removed C18: 10µF, SparkFun-Capacitors:EIA6032-NOM
- removed J1: (no value), SparkFun-Connectors:2X5_PTH_SILK_.05
- removed JP1, JP2: (no value), adafruit:1X08-3.5MM
- removed LED3, RXLED, TXLED: (no value), led:CHIP-LED0603
- removed R17: 1k, SparkFun-Resistors:0603
- removed R18: 47k, SparkFun-Resistors:0603
- removed R20, R25: 330, rcl:R0603
- removed S2: (no value), SparkFun-Switches:TACTILE_SWITCH_PTH_6.0MM
- removed U$5: MSP430FR2355, TTE:DA38
- removed U1: LTC1069-7CS8#PBF, TTE:SO-8_S
- removed U2: FT232RL-BASICSSOP, SparkFun:SSOP28DB
- added 1K: 1k, microbuilder:0805
- added 47K: 47k, microbuilder:0805
- added C1: 10µF, SparkFun-Capacitors:EIA6032-NOM
- added C2: 100nF, SparkFun-Capacitors:0805
- added C3: 22uF, SparkFun-Capacitors:0805
- added C4: 470n, SparkFun-Capacitors:0805
- added C5: .1u, SparkFun-Capacitors:0805
- added C6: 1n, SparkFun-Capacitors:0805
- added C7: 22p, SparkFun-Capacitors:0805
- added FILT: FILT, SparkFun-Connectors:1X02
- added FT232RL: FT232RL-BASICSSOP, SparkFun:SSOP28DB
- added GND, RXD, TCK, TDIO, TXD, VCC: 455-1750-1-ND, SparkFun-Connectors:1X04
- added J4, SIG: RX, SparkFun-Connectors:1X02
- added MSP430: MSP430FR2355, TTE:DA38
- added R2, R6: 330, microbuilder:0805
- added R4: 1M, SparkFun-Resistors:0603
- added RST: (no value), SparkFun-Switches:TACTILE_SWITCH_PTH_6.0MM
- added RX, STATUS, TX: (no value), microbuilder:CHIPLED_0805
- added TL069: LTC1069-7CS8#PBF, TTE:SO-8_S
- TM2: value (none) -> 100
- moved J2 100.2 mm to (36.8, -5.08)
- moved TM2 92.5 mm to (21.4, 31.6), turned to 270 degrees
- moved D1 92.3 mm to (26.9, 41.7), turned to 90 degrees
- moved RIGHT_ANGLE_SMA_MALE 59.0 mm to (21.3, 40.1), turned to 90 degrees
Connections:
- removed net !RTS!_JTAG_TCK: J1.7, U$5.8, U2.3
- removed net JTAG_TCK: J1.4, U$5.31
- removed net RESET_JTAG_RESET: C17.1, J1.10, R18.1, S2.3, U$5.9, U2.2
- removed net RX_INPUT_DAC_JTAG_TMS: J1.2, JP1.5, JP2.5
- removed net UART_BSL_RX_JTAG_DIN: J1.8, JP1.3, JP2.3, U$5.21, U$5.29, U2.1
- removed net UART_BSL_TX_JTAG_DOUT: J1.6, JP1.4, JP2.4, U$5.20, U$5.28, U2.5
- removed net VCC_3V3: U2.17, U2.4
- new net BCLUART_RXD: MSP430.21, MSP430.29, RXD.2
- new net BCLUART_RXD_EXT: RXD.3, RXD.4
- new net BCLUART_RXD_USB: FT232RL.1, RXD.1
- new net BCLUART_TXD: MSP430.20, MSP430.28, TXD.2
- new net BCLUART_TXD_EXT: TXD.3, TXD.4
- new net BCLUART_TXD_USB: FT232RL.5, TXD.1
- new net GND_EXT: GND.3, GND.4
- new net GND_USB: GND.1
- new net N$2: C7.2, TM2.2
- new net RST/SBWTDIO: 47K.1, C6.1, MSP430.9, RST.3, TDIO.2
- new net RST/SBWTDIO_EXT: TDIO.3, TDIO.4
- new net RST/SBWTDIO_USB: FT232RL.2, TDIO.1
- new net TEST/SSBWTCK: MSP430.8, TCK.2
- new net TEST/SSBWTCK_USB: FT232RL.3, TCK.1
- new net TST/SBWTCK_EXT: TCK.3, TCK.4
- new net VCC_EXT: VCC.3, VCC.4
- new net VCC_USB: FT232RL.17, FT232RL.4, VCC.1
- net ADC: now also J4.2, MSP430.5, MSP430.6; no longer U$5.5, U$5.6
- net ANTENNA_SIG: now also MSP430.38, R4.1, SIG.1; no longer JP1.8, JP2.8, U$5.38
- net ANTENNA_TX_SIG: now also C7.1, MSP430.34, SIG.2; no longer TM2.2, U$5.34
- net FILTER_CLK: now also 1K.1, MSP430.26; no longer R17.1, U$5.26
- net FILTER_IN: now also FILT.2, MSP430.30, MSP430.37, TL069.4; no longer JP1.6, JP2.6, U$5.30, U1.4
- net FILTER_OUT: now also FILT.1, MSP430.32, TL069.8; no longer JP1.7, JP2.7, U$5.32, U1.8
- net GND: now also C1.C, C2.2, C3.2, C4.1, C5.1, C6.2, FT232RL.18, FT232RL.21, FT232RL.25, FT232RL.26, FT232RL.7, GND.2, MSP430.11, R4.2, RIGHT_ANGLE_SMA_MALE.2, RIGHT_ANGLE_SMA_MALE.3, RIGHT_ANGLE_SMA_MALE.4, RIGHT_ANGLE_SMA_MALE.5, RST.1, STATUS.C, TL069.3, TL069.6, TL069.7; no longer C13.2, C14.2, C15.1, C16.1, C17.2, C18.C, J1.3, J1.5, J1.9, JP1.2, JP2.2, LED3.C, S2.1, U$5.11, U1.3, U1.6, U1.7, U2.18, U2.21, U2.25, U2.26, U2.7
- net N$1: now also 1K.2, TL069.5; no longer R17.2, U1.5
- net N$19: now also R2.1, STATUS.A; no longer LED3.A, R20.1
- net N$20: now also FT232RL.22, RX.C; no longer RXLED.C, U2.22
- net N$21: now also FT232RL.23, TX.C; no longer TXLED.C, U2.23
- net N$22: now also R6.1, RX.A, TX.A; no longer R25.1, RXLED.A, TXLED.A
- net N$3: now also C4.2, TL069.1; no longer C15.2, U1.1
- net P3.0/MCLK: now also MSP430.3; no longer U$5.3
- net P3.6/OA3-: now also MSP430.33; no longer U$5.33
- net RX_PGA_1: now also J4.1, MSP430.2, MSP430.4; no longer U$5.2, U$5.4
- net STATUS_LED: now also MSP430.15, R2.2; no longer R20.2, U$5.15
- net USB_DATA_+: now also FT232RL.15; no longer U2.15
- net USB_DATA_-: now also FT232RL.16; no longer U2.16
- net VCC: now also 47K.2, C1.A, C2.1, C3.1, C5.2, MSP430.10, R6.2, TL069.2, VCC.2; no longer C13.1, C14.1, C16.2, C18.A, J1.1, R18.2, R25.2, U$5.10, U1.2
- net V_USB: now also FT232RL.20; no longer JP1.1, JP2.1, U2.20
Routing:
- net GND1: track 0.00 -> 0.78 mm, vias 0 -> 1
- added copper zone on layer 1, net GND
- added copper zone on layer 16, net GND
Other:
- board size 100 x 80 mm -> 39.9 x 45.3 mm
- board text added: "FR2355"
- board text added: "I"
- board text added: "LTC1069"
- board text added: "O"
- board text added: "Rory Hancock - Blake Stadnyk Brody Dunlop - David Lutzer"
- board text added: "SIG"
- board text added: "TTE-Boys ECE Capstone 2019"
